Commit message: Task 1.1.3: Updated Origin in URDF

File: urdf/conveyor_belt.urdf (robot description, URDF)
Before this commit: robot conveyor_belt, 3 links, 2 joints
Joints:
- joint belt_body_joint: origin xyz=0.55656 -0.80919 0.80126 rpy=1.5708 0 0 -> xyz=0.05 0 0.25 rpy=0 0 0
- joint belt_moving_joint: origin xyz=-0.3981 0.1 0 rpy=0 0 0 -> xyz=0.0031673 0 0.1 rpy=0 0 0
