Commit message: Complete Setup

File: urdf/box.urdf.xacro (robot description, xacro)
@@ -3,10 +3,10 @@
      Commit Version: 1.6.0-4-g7f85cfe  Build Version: 1.6.7995.38578
      For more information, please see http://wiki.ros.org/sw_urdf_exporter -->
-<robot  name="conveyor_belt" xmlns:xacro="http://ros.org/wiki/xacro">
+<robot  name="box" xmlns:xacro="http://ros.org/wiki/xacro">
   <xacro:macro name="body_color">
     <visual>
       <material>
-        <ambient>0.501960784313725 0.501960784313725 0.501960784313725 1</ambient>
-        <diffuse>0.501960784313725 0.501960784313725 0.501960784313725 1</diffuse>
+        <ambient>0.909803921568627 0.443137254901961 0.0313725490196078 1</ambient>
+        <diffuse>0.909803921568627 0.443137254901961 0.0313725490196078 1</diffuse>
         <specular>0.1 0.1 0.1 1</specular>
         <emissive>0 0 0 0</emissive>
@@ -14,5 +14,5 @@
     </visual>
   </xacro:macro>
-  <xacro:macro name="belt_color">
+  <xacro:macro name="lid_color">
     <visual>
       <material>
@@ -28,15 +28,15 @@
     <inertial>
       <origin
-        xyz="1.15972439062802E-17 -0.0273162100367329 1.02144955943776E-17"
+        xyz="0.0182912425811423 0.00816214167781482 -0.0151972780093956"
         rpy="0 0 0" />
       <mass
-        value="2430.68583470577" />
+        value="0.5" />
       <inertia
-        ixx="431.198140853202"
-        ixy="2.18658245479853E-14"
-        ixz="4.38017677684144E-14"
-        iyy="7514.31711977665"
-        iyz="3.72364768160213E-15"
-        izz="7545.20095484556" />
+        ixx="0.405"
+        ixy="0"
+        ixz="0"
+        iyy="0.405"
+        iyz="0"
+        izz="0.405" />
     </inertial>
     <visual>
@@ -46,10 +46,10 @@
       <geometry>
         <mesh
-          filename="package://conveyor_belt/meshes/base_link.STL" />
+          filename="package://conveyor_belt/meshes/box/base_link.STL" />
       </geometry>
       <material
         name="">
         <color
-          rgba="0.501960784313725 0.501960784313725 0.501960784313725 1" />
+          rgba="0.909803921568627 0.443137254901961 0.0313725490196078 1" />
       </material>
     </visual>
@@ -60,23 +60,23 @@
       <geometry>
         <mesh
-          filename="package://conveyor_belt/meshes/base_link.STL" />
+          filename="package://conveyor_belt/meshes/box/base_link.STL" />
       </geometry>
     </collision>
   </link>
   <link
-    name="belt_link">
+    name="lid_link">
     <inertial>
       <origin
-        xyz="2.84 0.00499999999999995 2.76334119905601E-17"
+        xyz="6.93889390390723E-18 0.0163138686131387 -8.67361737988404E-18"
         rpy="0 0 0" />
       <mass
-        value="56.8" />
+        value="0.1" />
       <inertia
-        ixx="4.73380666666667"
-        ixy="3.71142749699624E-34"
-        ixz="2.20830761084774E-15"
-        iyy="157.442026666667"
-        iyz="2.30486925841449E-19"
-        izz="152.709166666667" />
+        ixx="0.0191640620437957"
+        ixy="-2.42137678137086E-18"
+        ixz="-1.26432854677493E-34"
+        iyy="0.0373576000000001"
+        iyz="1.0703877748923E-18"
+        izz="0.0191640620437957" />
     </inertial>
     <visual>
@@ -86,5 +86,5 @@
       <geometry>
         <mesh
-          filename="package://conveyor_belt/meshes/belt_link.STL" />
+          filename="package://conveyor_belt/meshes/box/lid_link.STL" />
       </geometry>
       <material
@@ -100,38 +100,27 @@
       <geometry>
         <mesh
-          filename="package://conveyor_belt/meshes/belt_link.STL" />
+          filename="package://conveyor_belt/meshes/box/lid_link.STL" />
       </geometry>
     </collision>
   </link>
   <joint
-    name="belt_joint"
-    type="prismatic">
+    name="lid_joint"
+    type="fixed">
     <origin
-      xyz="-2.83 0 0.3"
-      rpy="1.5708 0 0" />
+      xyz="0.018291 0.015197 0.16816"
+      rpy="-1.5708 0 3.1416" />
     <parent
       link="base_link" />
     <child
-      link="belt_link" />
+      link="lid_link" />
     <axis
-      xyz="-1 0 0" />
-    <limit
-      lower="0"
-      upper="0.01"
-      effort="0"
-      velocity="10" />
+      xyz="0 0 0" />
   </joint>
-<!-- Gazebo Colors -->
+  <!-- Gazebo Colors -->
   <gazebo reference="base_link">
     <xacro:body_color />
   </gazebo>
-  <gazebo reference="belt_link">
-    <xacro:belt_color />
-  </gazebo>
-<!-- Custom Gazebo Plugin for Conveyor Belt  -->
-  <gazebo>
-  <plugin filename="libconveyor_belt_plugin.so" name="conveyor_belt_plugin">
-        <max_velocity>0.3</max_velocity>
-  </plugin>
+  <gazebo reference="lid_link">
+    <xacro:lid_color />
   </gazebo>
 </robot>
